Commit message: feat: build mower model

File: urdf/mower_bot.xacro (robot description, xacro)
@@ -2,144 +2,189 @@
 <robot name="mower_bot" xmlns:xacro="http://www.ros.org/wiki/xacro">
   <xacro:include filename="$(find mower_bot)/urdf/mower_bot.gazebo" />
-  <xacro:property name="wheel_length" value="0.03" />
+  <!-- Length along X-axis, Width along Y-axis, Height along Z-axis -->
+  <xacro:property name="mower_width" value="0.4" />
+  <xacro:property name="mower_length" value="0.46" />
+  <xacro:property name="mower_height" value="0.3" />
+  <xacro:property name="mower_mass" value="8" />
+  <xacro:property name="base_x_offset" value="0" />
+  <xacro:property name="mower_inertia" value="${mower_mass/10.0}" />
+  <xacro:property name="mower_i_x_pos" value="${wheel_x_offset + mower_length/3.0}" />
+  <xacro:property name="mower_i_z_pos" value="${mower_height/10.0}" />
+  <xacro:property name="mower_frame_width" value="${mower_width - 2.1 * wheel_length}" />
+  <xacro:property name="mower_frame_length" value="${mower_length*1.2}" />
+  <xacro:property name="mower_frame_height" value="${mower_height/4.0}" />
+  <xacro:property name="hardware_width" value="${mower_width/2.0}" />
+  <xacro:property name="hardware_length" value="${mower_length/2.0}" />
+  <xacro:property name="hardware_height" value="${mower_height/2.0}" />
+  <xacro:property name="hardware_z_offset" value="${hardware_height/2.0}" />
+  <xacro:property name="wheel_length" value="0.05" />
   <xacro:property name="wheel_radius" value="0.08" />
-  <xacro:property name="wheel_mass" value="0.5" />
+  <xacro:property name="wheel_mass" value="1" />
   <xacro:property name="wheel_inertia" value="1e-3" />
-  <xacro:property name="cutter_radius" value="0.16" />
-  <xacro:property name="cutter_height" value="0.08" />
-  <xacro:property name="motor_height" value="0.16" />
-  <xacro:property name="motor_length" value="0.15" />
-  <xacro:property name="motor_width" value="0.2" />
-  <xacro:property name="motor_z_offset" value="${cutter_height + motor_height/2.0 - 0.04}" />
-  <xacro:property name="cutter_mass" value="10" />
-  <xacro:property name="cutter_inertia" value="0.1" />
-  <xacro:property name="chassis_length" value="0.26" />
-  <xacro:property name="chassis_depth" value="0.04" />
-  <xacro:property name="chassis_mass" value="15" />
-  <xacro:property name="chassis_inertia" value="0.01" />
-  <xacro:property name="chassis_long_width" value="${2.0*cutter_radius + 2.0*chassis_depth}" />
-  <xacro:property name="chassis_x_offset" value="${cutter_radius + 0.02}" />
-  <xacro:property name="chassis_y_offset" value="${chassis_length/2.0 - chassis_depth/2.0}" />
-  <xacro:property name="chassis_z_offset" value="${cutter_height - chassis_depth}" />
-  <xacro:property name="cutter_height_offset" value="0.03" />
-  <xacro:property name="wheel_x_offset" value="${chassis_x_offset}" />
-  <xacro:property name="wheel_y_offset" value="${chassis_length/2.0 + wheel_length/2.0 + 0.002}" />
-  <xacro:property name="laser_z_offset" value="${motor_z_offset + motor_height/2.0}" />
+  <xacro:property name="wheel_x_offset" value="${base_x_offset - mower_length/2.0}" />
+  <xacro:property name="wheel_y_offset" value="${mower_width/2.0 - wheel_length/2.0}" />
+  <xacro:property name="caster_radius" value="${wheel_radius/2.0}" />
+  <xacro:property name="caster_x_offset" value="${base_x_offset + mower_length/2.0}" />
+  <xacro:property name="caster_y_offset" value="${wheel_y_offset - 0.07}" />
+  <xacro:property name="caster_z_offset" value="${caster_radius}" />
+  <xacro:property name="camerra_width" value="0.05" />
+  <xacro:property name="camerra_length" value="0.05" />
+  <xacro:property name="camerra_height" value="0.05" />
+  <xacro:property name="camerra_x_offset" value="${hardware_length/2.0 + base_x_offset - camerra_length/2.0 + 0.001}" />
+  <xacro:property name="camerra_z_offset" value="${hardware_height - camerra_height/2.0 + 0.001}" />
+  <xacro:property name="laser_width" value="0.1" />
+  <xacro:property name="laser_length" value="0.1" />
+  <xacro:property name="laser_height" value="0.1" />
+  <xacro:property name="laser_x_offset" value="${base_x_offset}" />
+  <xacro:property name="laser_z_offset" value="${hardware_height + 0.025}" />
   <link name="robot_footprint"></link>
   <joint name="robot_footprint_joint" type="fixed">
     <origin xyz="0 0 0" rpy="0 0 0" />
-    <parent link="robot_footprint"/>
-    <child link="cutter" />
-  </joint>
-  <!-- blade cage -->
-  <link name='cutter'>
-    <inertial>
-      <mass value="${cutter_mass}"/>
-      <origin xyz="0 0 ${cutter_height_offset}" rpy=" 0 0 0"/>
-      <inertia
-          ixx="${cutter_inertia}" ixy="0" ixz="0"
-          iyy="${cutter_inertia}" iyz="0"
-          izz="${cutter_inertia}" />
-    </inertial>
-    <collision name='collision'>
-      <origin xyz="0 0 ${cutter_height_offset}" rpy=" 0 0 0"/>
-      <geometry>
-        <cylinder radius="${cutter_radius}" length="${cutter_height}"/>
+    <parent link="robot_footprint" />
+    <child link="chassis" />
+  </joint>
+  <link name='chassis'>
+    <inertial>
+      <mass value="${mower_mass}"/>
+      <origin xyz="${mower_i_x_pos} 0 ${mower_i_z_pos}" rpy=" 0 0 0"/>
+      <inertia
+          ixx="${mower_inertia}" ixy="0" ixz="0"
+          iyy="${mower_inertia}" iyz="0"
+          izz="${mower_inertia}" />
+    </inertial>
+    <collision>
+      <origin xyz="${base_x_offset} 0 0" rpy=" 0 0 0"/>
+      <geometry>
+        <box size="${mower_frame_length} ${mower_frame_width} ${mower_frame_height}"/>
       </geometry>
     </collision>
     <visual>
-      <origin xyz="0 0 ${cutter_height_offset}" rpy=" 0 0 0"/>
-      <geometry>
-        <cylinder radius="${cutter_radius}" length="${cutter_height}"/>
-      </geometry>
-    </visual>
+      <origin xyz="${base_x_offset} 0 0" rpy=" 0 0 0"/>
+      <geometry>
+        <box size="${mower_frame_length} ${mower_frame_width} ${mower_frame_height}"/>
+      </geometry>
+    </visual>
+    <!-- blade frame -->
     <collision>
-      <origin xyz="0 0 ${motor_z_offset}" rpy=" 0 0 0"/>
-      <geometry>
-        <box size="${chassis_depth} ${chassis_length} ${chassis_depth}"/>
+      <origin xyz="${base_x_offset} 0 0" rpy=" 0 0 0"/>
+      <geometry>
+        <cylinder radius="${mower_width/2.0}" length="${mower_frame_height}"/>
       </geometry>
     </collision>
     <visual>
-      <origin xyz="0 0 ${motor_z_offset}" rpy=" 0 0 0"/>
-      <geometry>
-        <box size="${motor_width} ${motor_length} ${motor_height}"/>
-      </geometry>
-    </visual>
-  </link>
-  <joint type="fixed" name="frame_connect">
-    <origin xyz="0 0 0" rpy="0 0 0"/>
-    <child link="chassis"/>
-    <parent link="cutter"/>
-    <axis xyz="0 1 0" rpy="0 0 0"/>
-    <limit effort="10000" velocity="1000"/>
-    <joint_properties damping="1.0" friction="1.0"/>
-  </joint>
-  <link name='chassis'>
-    <inertial>
-      <mass value="${chassis_mass}"/>
-      <origin xyz="0 0 0" rpy=" 0 0 0"/>
-      <inertia
-          ixx="${chassis_inertia}" ixy="0" ixz="0"
-          iyy="${chassis_inertia}" iyz="0"
-          izz="${chassis_inertia}" />
-    </inertial>
+      <origin xyz="${base_x_offset} 0 0" rpy=" 0 0 0"/>
+      <geometry>
+        <cylinder radius="${mower_width/2.0}" length="${mower_frame_height}"/>
+      </geometry>
+    </visual>
+    <!-- hardware frame -->
     <collision>
-      <origin xyz="${chassis_x_offset} 0 ${chassis_z_offset}" rpy=" 0 0 0"/>
-      <geometry>
-        <box size="${chassis_depth} ${chassis_length} ${chassis_depth}"/>
+      <origin xyz="${base_x_offset} 0 ${hardware_z_offset}" rpy=" 0 0 0"/>
+      <geometry>
+        <box size="${hardware_length} ${hardware_width} ${hardware_height}"/>
       </geometry>
     </collision>
     <visual>
-      <origin xyz="${chassis_x_offset} 0 ${chassis_z_offset}" rpy=" 0 0 0"/>
-      <geometry>
-        <box size="${chassis_depth} ${chassis_length} ${chassis_depth}"/>
-      </geometry>
-    </visual>
-    <collision>
-      <origin xyz="-${chassis_x_offset} 0 ${chassis_z_offset}" rpy=" 0 0 0"/>
-      <geometry>
-        <box size="${chassis_depth} ${chassis_length} ${chassis_depth}"/>
-      </geometry>
-    </collision>
-    <visual>
-      <origin xyz="-${chassis_x_offset} 0 ${chassis_z_offset}" rpy=" 0 0 0"/>
-      <geometry>
-        <box size="${chassis_depth} ${chassis_length} ${chassis_depth}"/>
-      </geometry>
-    </visual>
-    <collision>
-      <origin xyz="0 ${chassis_y_offset} ${chassis_z_offset}" rpy=" 0 0 0"/>
-      <geometry>
-        <box size="${chassis_length} ${chassis_depth}  ${chassis_depth}"/>
-      </geometry>
-    </collision>
-    <visual>
-      <origin xyz="0 ${chassis_y_offset} ${cutter_height}" rpy=" 0 0 0"/>
-      <geometry>
-        <box size="${chassis_long_width} ${chassis_depth}  ${chassis_depth}"/>
-      </geometry>
-    </visual>
-    <collision>
-      <origin xyz="0 -${chassis_y_offset} ${chassis_z_offset}" rpy=" 0 0 0"/>
-      <geometry>
-        <box size="${chassis_length} ${chassis_depth}  ${chassis_depth}"/>
-      </geometry>
-    </collision>
-    <visual>
-      <origin xyz="0 -${chassis_y_offset} ${cutter_height}" rpy=" 0 0 0"/>
-      <geometry>
-        <box size="${chassis_long_width} ${chassis_depth}  ${chassis_depth}"/>
-      </geometry>
-    </visual>
-  </link>
-  <joint type="continuous" name="right_back_wheel_hinge">
-    <origin xyz="-${wheel_x_offset} -${wheel_y_offset} ${chassis_z_offset}" rpy="0 0 0"/>
-    <child link="right_back_wheel"/>
-    <parent link="chassis"/>
-    <axis xyz="0 1 0" rpy="0 0 0"/>
-    <limit effort="10000" velocity="1000"/>
-    <joint_properties damping="1.0" friction="1.0"/>
-  </joint>
-  <link name="right_back_wheel">
+      <origin xyz="${base_x_offset} 0 ${hardware_z_offset}" rpy=" 0 0 0"/>
+      <geometry>
+        <box size="${hardware_length} ${hardware_width} ${hardware_height}"/>
+      </geometry>
+    </visual>
+    <collision name='left_caster_collision'>
+      <origin xyz="${caster_x_offset} ${caster_y_offset} -${caster_z_offset}" rpy=" 0 0 0"/>
+      <geometry>
+        <sphere radius="${caster_radius}"/>
+      </geometry>
+      <surface>
+        <friction>
+          <ode>
+            <mu>0</mu>
+            <mu2>0</mu2>
+            <slip1>1.0</slip1>
+            <slip2>1.0</slip2>
+          </ode>
+        </friction>
+      </surface>
+    </collision>
+    <visual name='left_caster_visual'>
+      <origin xyz="${caster_x_offset} ${caster_y_offset} -${caster_z_offset}" rpy=" 0 0 0"/>
+      <geometry>
+        <sphere radius="${caster_radius}"/>
+      </geometry>
+    </visual>
+    <collision name='right_caster_collision'>
+      <origin xyz="${caster_x_offset} -${caster_y_offset} -${caster_z_offset}" rpy=" 0 0 0"/>
+      <geometry>
+        <sphere radius="${caster_radius}"/>
+      </geometry>
+      <surface>
+        <friction>
+          <ode>
+            <mu>0</mu>
+            <mu2>0</mu2>
+            <slip1>1.0</slip1>
+            <slip2>1.0</slip2>
+          </ode>
+        </friction>
+      </surface>
+    </collision>
+    <visual name='right_caster_visual'>
+      <origin xyz="${caster_x_offset} -${caster_y_offset} -${caster_z_offset}" rpy=" 0 0 0"/>
+      <geometry>
+        <sphere radius="${caster_radius}"/>
+      </geometry>
+    </visual>
+  </link>
+  <!-- left wheel -->
+  <joint type="continuous" name="left_wheel_hinge">
+    <origin xyz="${wheel_x_offset} ${wheel_y_offset} 0" rpy="0 0 0"/>
+    <child link="left_wheel"/>
+    <parent link="chassis"/>
+    <axis xyz="0 1 0" rpy="0 0 0"/>
+    <limit effort="10000" velocity="1000"/>
+    <joint_properties damping="1.0" friction="1.0"/>
+  </joint>
+  <link name="left_wheel">
+    <inertial>
+      <mass value="${wheel_mass}"/>
+      <origin xyz="0.0 0 0" rpy=" 0 1.5707 1.5707"/>
+      <inertia
+        ixx="${wheel_inertia}" ixy="0" ixz="0"
+        iyy="${wheel_inertia}" iyz="0"
+        izz="${wheel_inertia}" />
+    </inertial>
+    <collision name="left_wheel_collision">
+      <origin xyz="0 0 0" rpy=" 0 1.5707 1.5707"/>
+      <geometry>
+        <cylinder length="${wheel_length}" radius="${wheel_radius}"/>
+      </geometry>
+      <surface>
+        <friction>
+          <ode>
+            <mu>100</mu>
+            <mu2>100</mu2>
+            <slip1>0</slip1>
+            <slip2>0</slip2>
+          </ode>
+        </friction>
+      </surface>
+    </collision>
+    <visual name="left_wheel_visual">
+      <origin xyz="0 0 0" rpy=" 0 1.5707 1.5707"/>
+      <geometry>
+        <cylinder length="${wheel_length}" radius="${wheel_radius}"/>
+      </geometry>
+    </visual>
+  </link>
+  <!-- right wheel -->
+  <joint type="continuous" name="right_wheel_hinge">
+    <origin xyz="${wheel_x_offset} -${wheel_y_offset} 0" rpy="0 0 0"/>
+    <child link="right_wheel"/>
+    <parent link="chassis"/>
+    <axis xyz="0 1 0" rpy="0 0 0"/>
+    <limit effort="10000" velocity="1000"/>
+    <joint_properties damping="1.0" friction="1.0"/>
+  </joint>
+  <link name="right_wheel">
     <inertial>
       <mass value="${wheel_mass}"/>
@@ -150,120 +195,31 @@
           izz="${wheel_inertia}" />
     </inertial>
-    <collision name="collision">
-      <origin xyz="0 0 0" rpy=" 0 1.5707 1.5707"/>
-      <geometry>
-        <cylinder length="${wheel_length}" radius="${wheel_radius}"/>
-      </geometry>
-    </collision>
-    <visual>
-      <origin xyz="0 0 0" rpy=" 0 1.5707 1.5707"/>
-      <geometry>
-        <cylinder length="${wheel_length}" radius="${wheel_radius}"/>
-      </geometry>
-    </visual>
-  </link>
-  <joint type="continuous" name="left_back_wheel_hinge">
-    <origin xyz="-${wheel_x_offset} ${wheel_y_offset} ${chassis_z_offset}" rpy="0 0 0"/>
-    <child link="left_back_wheel"/>
-    <parent link="chassis"/>
-    <axis xyz="0 1 0" rpy="0 0 0"/>
-    <limit effort="10000" velocity="1000"/>
-    <joint_properties damping="1.0" friction="1.0"/>
-  </joint>
-  <link name="left_back_wheel">
-    <inertial>
-      <mass value="${wheel_mass}"/>
-      <origin xyz="0.0 0 0" rpy=" 0 1.5707 1.5707"/>
-      <inertia
-          ixx="${wheel_inertia}" ixy="0" ixz="0"
-          iyy="${wheel_inertia}" iyz="0"
-          izz="${wheel_inertia}" />
-    </inertial>
-    <collision name="collision">
-      <origin xyz="0 0 0" rpy=" 0 1.5707 1.5707"/>
-      <geometry>
-        <cylinder length="${wheel_length}" radius="${wheel_radius}"/>
-      </geometry>
-    </collision>
-    <visual>
-      <origin xyz="0 0 0" rpy=" 0 1.5707 1.5707"/>
-      <geometry>
-        <cylinder length="${wheel_length}" radius="${wheel_radius}"/>
-      </geometry>
-    </visual>
-  </link>
-  <joint type="continuous" name="right_front_wheel_hinge">
-    <origin xyz="${wheel_x_offset} -${wheel_y_offset} ${chassis_z_offset}" rpy="0 0 0"/>
-    <child link="right_front_wheel"/>
-    <parent link="chassis"/>
-    <axis xyz="0 1 0" rpy="0 0 0"/>
-    <limit effort="10000" velocity="1000"/>
-    <joint_properties damping="1.0" friction="1.0"/>
-  </joint>
-  <link name="right_front_wheel">
-    <inertial>
-      <mass value="${wheel_mass}"/>
-      <origin xyz="0.0 0 0" rpy=" 0 1.5707 1.5707"/>
-      <inertia
-          ixx="${wheel_inertia}" ixy="0" ixz="0"
-          iyy="${wheel_inertia}" iyz="0"
-          izz="${wheel_inertia}" />
-    </inertial>
-    <collision name="collision">
-      <origin xyz="0 0 0" rpy=" 0 1.5707 1.5707"/>
-      <geometry>
-        <cylinder length="${wheel_length}" radius="${wheel_radius}"/>
-      </geometry>
-    </collision>
-    <visual>
-      <origin xyz="0 0 0" rpy=" 0 1.5707 1.5707"/>
-      <geometry>
-        <cylinder length="${wheel_length}" radius="${wheel_radius}"/>
-      </geometry>
-    </visual>
-  </link>
-  <joint type="continuous" name="left_front_wheel_hinge">
-    <origin xyz="${wheel_x_offset} ${wheel_y_offset} ${chassis_z_offset}" rpy="0 0 0"/>
-    <child link="left_front_wheel"/>
-    <parent link="chassis"/>
-    <axis xyz="0 1 0" rpy="0 0 0"/>
-    <limit effort="10000" velocity="1000"/>
-    <joint_properties damping="1.0" friction="1.0"/>
-  </joint>
-  <link name="left_front_wheel">
-    <inertial>
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
Commit message: Feat: add scale factor to model

File: urdf/mower_bot.xacro (robot description, xacro)
@@ -2,9 +2,11 @@
 <robot name="mower_bot" xmlns:xacro="http://www.ros.org/wiki/xacro">
   <xacro:include filename="$(find mower_bot)/urdf/mower_bot.gazebo" />
+  <!-- Scale the robot size to fit the environment -->
+  <xacro:property name="scale" value="1.25" />
   <!-- Length along X-axis, Width along Y-axis, Height along Z-axis -->
-  <xacro:property name="mower_width" value="0.4" />
-  <xacro:property name="mower_length" value="0.46" />
-  <xacro:property name="mower_height" value="0.3" />
-  <xacro:property name="mower_mass" value="8" />
+  <xacro:property name="mower_width" value="${scale * 0.5}" />
+  <xacro:property name="mower_length" value="${scale * 0.5}" />
+  <xacro:property name="mower_height" value="${scale * 0.3}" />
+  <xacro:property name="mower_mass" value="${scale * 8}" />
   <xacro:property name="base_x_offset" value="0" />
   <xacro:property name="mower_inertia" value="${mower_mass/10.0}" />
@@ -18,8 +20,8 @@
   <xacro:property name="hardware_height" value="${mower_height/2.0}" />
   <xacro:property name="hardware_z_offset" value="${hardware_height/2.0}" />
-  <xacro:property name="wheel_length" value="0.05" />
-  <xacro:property name="wheel_radius" value="0.08" />
-  <xacro:property name="wheel_mass" value="1" />
-  <xacro:property name="wheel_inertia" value="1e-3" />
+  <xacro:property name="wheel_length" value="${scale * 0.05}" />
+  <xacro:property name="wheel_radius" value="${scale * 0.08}" />
+  <xacro:property name="wheel_mass" value="${scale * 1}" />
+  <xacro:property name="wheel_inertia" value="${scale * 1e-3}" />
   <xacro:property name="wheel_x_offset" value="${base_x_offset - mower_length/2.0}" />
   <xacro:property name="wheel_y_offset" value="${mower_width/2.0 - wheel_length/2.0}" />
@@ -159,14 +161,4 @@
         <cylinder length="${wheel_length}" radius="${wheel_radius}"/>
       </geometry>
-      <surface>
-        <friction>
-          <ode>
-            <mu>100</mu>
-            <mu2>100</mu2>
-            <slip1>0</slip1>
-            <slip2>0</slip2>
-          </ode>
-        </friction>
-      </surface>
     </collision>
     <visual name="left_wheel_visual">
@@ -200,14 +192,4 @@
         <cylinder length="${wheel_length}" radius="${wheel_radius}"/>
       </geometry>
-      <surface>
-        <friction>
-          <ode>
-            <mu>100</mu>
-            <mu2>100</mu2>
-            <slip1>0</slip1>
-            <slip2>0</slip2>
-          </ode>
-        </friction>
-      </surface>
     </collision>
     <visual name="right_wheel_visual">

Commit message: Change: variable values

File: urdf/mower_bot.xacro (robot description, xacro)
@@ -3,13 +3,13 @@
   <xacro:include filename="$(find mower_bot)/urdf/mower_bot.gazebo" />
   <!-- Scale the robot size to fit the environment -->
-  <xacro:property name="scale" value="1.25" />
+  <xacro:property name="scale" value="1.0" />
   <!-- Length along X-axis, Width along Y-axis, Height along Z-axis -->
-  <xacro:property name="mower_width" value="${scale * 0.5}" />
-  <xacro:property name="mower_length" value="${scale * 0.5}" />
+  <xacro:property name="mower_width" value="${scale * 0.36}" />
+  <xacro:property name="mower_length" value="${scale * 0.46}" />
   <xacro:property name="mower_height" value="${scale * 0.3}" />
   <xacro:property name="mower_mass" value="${scale * 8}" />
   <xacro:property name="base_x_offset" value="0" />
   <xacro:property name="mower_inertia" value="${mower_mass/10.0}" />
-  <xacro:property name="mower_i_x_pos" value="${wheel_x_offset + mower_length/3.0}" />
+  <xacro:property name="mower_i_x_pos" value="${wheel_x_offset + mower_length/3.0}" /> -->
   <xacro:property name="mower_i_z_pos" value="${mower_height/10.0}" />
   <xacro:property name="mower_frame_width" value="${mower_width - 2.1 * wheel_length}" />

Commit message: chore: calculates inertia

File: urdf/mower_bot.xacro (robot description, xacro)
@@ -10,6 +10,12 @@
   <xacro:property name="mower_mass" value="${scale * 8}" />
   <xacro:property name="base_x_offset" value="0" />
-  <xacro:property name="mower_inertia" value="${mower_mass/10.0}" />
-  <xacro:property name="mower_i_x_pos" value="${wheel_x_offset + mower_length/3.0}" /> -->
+  <!-- inertia = 1/12*m(h^2+d^2) -->
+  <xacro:property name="height_2" value="${mower_height * mower_height}" />
+  <xacro:property name="width_2" value="${mower_width * mower_width}" />
+  <xacro:property name="length_2" value="${mower_length * mower_length}" />
+  <xacro:property name="mower_inertia_xx" value="${mower_mass/12.0 * (height_2 + width_2)}" />
+  <xacro:property name="mower_inertia_yy" value="${mower_mass/12.0 * (height_2 + length_2)}" />
+  <xacro:property name="mower_inertia_zz" value="${mower_mass/12.0 * (width_2 + length_2)}" />
+  <xacro:property name="mower_i_x_pos" value="${wheel_x_offset + mower_length/3.0}" />
   <xacro:property name="mower_i_z_pos" value="${mower_height/10.0}" />
   <xacro:property name="mower_frame_width" value="${mower_width - 2.1 * wheel_length}" />
@@ -51,7 +57,7 @@
       <origin xyz="${mower_i_x_pos} 0 ${mower_i_z_pos}" rpy=" 0 0 0"/>
       <inertia
-          ixx="${mower_inertia}" ixy="0" ixz="0"
-          iyy="${mower_inertia}" iyz="0"
-          izz="${mower_inertia}" />
+          ixx="${mower_inertia_xx}" ixy="0" ixz="0"
+          iyy="${mower_inertia_yy}" iyz="0"
+          izz="${mower_inertia_zz}" />
     </inertial>
     <collision>
@@ -161,4 +167,14 @@
         <cylinder length="${wheel_length}" radius="${wheel_radius}"/>
       </geometry>
+      <surface>
+        <friction>
+          <ode>
+            <mu>1</mu>
+            <mu2>1</mu2>
+            <slip1>0.5</slip1>
+            <slip2>0</slip2>
+          </ode>
+        </friction>
+      </surface>
     </collision>
     <visual name="left_wheel_visual">
@@ -192,4 +208,14 @@
         <cylinder length="${wheel_length}" radius="${wheel_radius}"/>
       </geometry>
+      <surface>
+        <friction>
+          <ode>
+            <mu>1</mu>
+            <mu2>1</mu2>
+            <slip1>0.5</slip1>
+            <slip2>0</slip2>
+          </ode>
+        </friction>
+      </surface>
     </collision>
     <visual name="right_wheel_visual">
