Commit message: Chore: rename model to skid_steer_bot

File: urdf/skid_steer_bot.xacro (robot description, xacro)
@@ -1,5 +1,5 @@
 <?xml version='1.0'?>
-<robot name="mower_bot" xmlns:xacro="http://www.ros.org/wiki/xacro">
-  <xacro:include filename="$(find mower_bot)/urdf/mower_bot.gazebo" />
+<robot name="skid_steer_bot" xmlns:xacro="http://www.ros.org/wiki/xacro">
+  <xacro:include filename="$(find skid_steer_bot)/urdf/skid_steer_bot.gazebo" />
   <!-- Scale the robot size to fit the environment -->
   <xacro:property name="scale" value="1.0" />
@@ -319,5 +319,5 @@
       <origin xyz="0 0 0" rpy=" 0 0 0"/>
       <geometry>
-        <mesh filename="package://mower_bot/meshes/hokuyo.dae"/>
+        <mesh filename="package://skid_steer_bot/meshes/hokuyo.dae"/>
       </geometry>
     </visual>

Commit message: feat: parameter update for submit

File: urdf/skid_steer_bot.xacro (robot description, xacro)
@@ -8,5 +8,5 @@
   <xacro:property name="mower_length" value="${scale * 0.46}" />
   <xacro:property name="mower_height" value="${scale * 0.3}" />
-  <xacro:property name="mower_mass" value="${scale * 8}" />
+  <xacro:property name="mower_mass" value="${scale * 10}" />
   <xacro:property name="base_x_offset" value="0" />
   <!-- inertia = 1/12*m(h^2+d^2) -->
